Commit message: - URDF file is completed. - Spawn the robot in gazebo is completed. - Launch file to start robot in gazebo created. - Fix the colors with gazebo material is done.

File: My-ROS2-Humble/Tutorial_MobileRobot/mobilebot_ws/install/mobilebot_description/share/mobilebot_description/urdf/common_properties.xacro (robot description, xacro)
@@ -10,3 +10,30 @@
         <color rgba="0.5 0 0 1"/>
     </material>
+    <xacro:macro name="box_inertia" params="mass length width height xyz rpy">
+        <inertial>
+            <origin xyz="${xyz}" rpy="${rpy}"/>
+            <mass value="${mass}"/>
+            <inertia ixx="${(mass/12) * (height*height + length*length)}" ixy="0" ixz="0"
+                     iyy="${(mass/12) * (width*width + length*length)}" iyz="0"
+                     izz="${(mass/12) * (width*width + height*height)}"/>
+        </inertial>
+    </xacro:macro>
+    <xacro:macro name="cylinder_inertia" params="mass radius height xyz rpy">
+        <inertial>
+            <origin xyz="${xyz}" rpy="${rpy}"/>
+            <mass value="${mass}"/>
+            <inertia ixx="${(mass/12) * (3*radius*radius + height*height)}" ixy="0" ixz="0"
+                     iyy="${(mass/12) * (3*radius*radius + height*height)}" iyz="0"
+                     izz="${(mass/2) * (radius*radius)}"/>
+        </inertial>
+    </xacro:macro>
+    <xacro:macro name="sphere_inertia" params="mass radius xyz rpy">
+        <inertial>
+            <origin xyz="${xyz}" rpy="${rpy}"/>
+            <mass value="${mass}"/>
+            <inertia ixx="${(2/5) * mass * radius*radius}" ixy="0" ixz="0"
+                     iyy="${(2/5) * mass * radius*radius}" iyz="0"
+                     izz="${(2/5) * mass * radius*radius}"/>
+        </inertial>
+    </xacro:macro>
 </robot>

File: My-ROS2-Humble/Tutorial_MobileRobot/mobilebot_ws/install/mobilebot_description/share/mobilebot_description/urdf/mobilebot.urdf.xacro (robot description, xacro)
@@ -4,3 +4,4 @@
     <xacro:include filename="common_properties.xacro"/>
     <xacro:include filename="mobilebot_base.xacro"/>
+    <xacro:include filename="mobilebot_base_gazebo.xacro"/>
 </robot>

File: My-ROS2-Humble/Tutorial_MobileRobot/mobilebot_ws/install/mobilebot_description/share/mobilebot_description/urdf/mobilebot_base.xacro (robot description, xacro)
@@ -1,5 +1,5 @@
 <?xml version="1.0"?>
 <robot xmlns:xacro="http://www.ros.org/wiki/xacro">
-    <!-- xacro defines -->
+    <!-- #### ##### xacro defines ##### #### -->
     <xacro:property name="PI"           value="3.14159"/>
     <xacro:property name="base_length"  value="0.6"/>
@@ -8,5 +8,29 @@
     <xacro:property name="wheel_radius" value="0.1"/>
     <xacro:property name="wheel_length" value="0.05"/>
-    <!-- xacro functions -->
+    <!-- #### ##### Base Link and Base footprint ##### #### -->
+    <link name="base_footprint"/>
+    <link name="base_link">
+        <visual>    <!-- give a shape to it -->
+             <geometry>
+                <box size="${base_length} ${base_width} ${base_height}"/>   <!-- 60cm length, 40cm width, 20cm height-->
+             </geometry>
+             <origin xyz="0 0 ${base_height/2}" rpy="0 0 0"/>
+             <material name="blue"/>
+        </visual>
+        <collision>
+            <geometry>
+                <box size="${base_length} ${base_width} ${base_height}"/>   <!-- 60cm length, 40cm width, 20cm height-->
+             </geometry>
+             <origin xyz="0 0 ${base_height/2}" rpy="0 0 0"/>
+        </collision>
+        <xacro:box_inertia mass="1.0" length="${base_length}" width="${base_width}" height="${base_height}"
+                            xyz="0 0 ${base_height/2}" rpy="0 0 0"/>
+    </link>
+    <joint name="footprint_BaseLink_joint" type="fixed">
+        <parent link="base_footprint"/>
+        <child link="base_link"/>
+        <origin xyz="0 0 ${wheel_radius}" rpy="0 0 0"/>
+    </joint>
+    <!-- #### ##### xacro functions ##### #### -->
     <xacro:macro name="wheel_link" params="prefix">
         <link name="${prefix}_wheel_link">
@@ -18,21 +42,15 @@
                 <material name="red"/>
             </visual>
+            <collision>
+                <geometry>
+                    <cylinder radius="${wheel_radius}" length="${wheel_length}"/>
+                </geometry>
+                <origin xyz="0 0 0" rpy="${PI/2} 0 0"/>     <!-- 90degree in X-Axis-->
+            </collision>
+            <xacro:cylinder_inertia mass="0.4" radius="${wheel_radius}" height="${wheel_length}"
+                                     xyz="0 0 0" rpy="${PI/2} 0 0"/>
         </link>
     </xacro:macro>
-    <link name="base_footprint"/>
-    <link name="base_link">
-        <visual>    <!-- give a shape to it -->
-             <geometry>
-                <box size="${base_length} ${base_width} ${base_height}"/>   <!-- 60cm length, 40cm width, 20cm height-->
-             </geometry>
-             <origin xyz="0 0 ${base_height/2}" rpy="0 0 0"/>
-             <material name="blue"/>
-        </visual>
-    </link>
-    <joint name="footprint_BaseLink_joint" type="fixed">
-        <parent link="base_footprint"/>
-        <child link="base_link"/>
-        <origin xyz="0 0 ${wheel_radius}" rpy="0 0 0"/>
-    </joint>
+    <!-- #### ##### Right Wheel Link ##### #### -->
     <xacro:wheel_link prefix="right"/>
     <joint name="base_RightWheel_joint" type="continuous">  <!-- continuous is a revolution with no limit-->
@@ -42,4 +60,5 @@
         <axis xyz="0 1 0"/> <!-- rotate on Y-Axis -->
     </joint>
+    <!-- #### ##### Left Wheel Link ##### #### -->
     <xacro:wheel_link prefix="left"/>
     <joint name="base_LeftWheel_joint" type="continuous">  <!-- continuous is a revolution with no limit-->
@@ -49,4 +68,5 @@
         <axis xyz="0 1 0"/> <!-- rotate on Y-Axis -->
     </joint>
+    <!-- #### ##### Caster Wheel Link ##### #### -->
     <link name="caster_wheel_link">
         <visual>
@@ -57,4 +77,12 @@
             <material name="red"/>
         </visual>
+        <collision>
+            <geometry>
+                <sphere radius="${wheel_radius/2}"/>
+            </geometry>
+            <origin xyz="0 0 0" rpy="0 0 0"/>
+        </collision>
+        <xacro:sphere_inertia mass="0.2" radius="${wheel_radius/2}"
+                              xyz="0 0 0" rpy="0 0 0"/>
     </link>
     <joint name="base_CasterWheel_joint" type="fixed">

Commit message: tutorial_project is completed

File: My-ROS2-Humble/Tutorial_MobileRobot/mobilebot_ws/install/mobilebot_description/share/mobilebot_description/urdf/common_properties.xacro (robot description, xacro)
@@ -9,4 +9,7 @@
     <material name="red">
         <color rgba="0.5 0 0 1"/>
+    </material>
+    <material name="orange">
+        <color rgba="1 0.3 0 1"/>
     </material>
     <xacro:macro name="box_inertia" params="mass length width height xyz rpy">

File: My-ROS2-Humble/Tutorial_MobileRobot/mobilebot_ws/install/mobilebot_description/share/mobilebot_description/urdf/mobilebot.urdf.xacro (robot description, xacro)
@@ -5,3 +5,11 @@
     <xacro:include filename="mobilebot_base.xacro"/>
     <xacro:include filename="mobilebot_base_gazebo.xacro"/>
+    <xacro:include filename="arm.xacro"/>
+    <xacro:include filename="arm_gazebo.xacro"/>
+    <!-- #### Combine the robot(mobilebot) and arm #### -->
+    <joint name="mobilebot_base_arm_joint" type="fixed">
+        <parent link="base_link"/>
+        <child link="arm_base_link"/>
+        <origin xyz="${base_length/4} 0 ${base_height}" rpy="0 0 0"/>
+    </joint>
 </robot>

File: My-ROS2-Humble/Tutorial_MobileRobot/mobilebot_ws/install/mobilebot_description/share/mobilebot_description/urdf/mobilebot_base_gazebo.xacro (robot description, xacro)
@@ -16,4 +16,5 @@
         <mu2 value="0.1"/>
     </gazebo>
+    <!-- #### Gazebo Plugins ##### -->
     <gazebo>
         <plugin name="diff_drive_controller" filename="libgazebo_ros_diff_drive.so">
