Commit message: feat: add diff drive and arm controllers configuration and implement MobileBase hardware interface
- Added diff_drive_controller and arm joint controller parameters
- Defined ros2_control hardware configuration for mobile base in URDF
- Implemented MobileBaseHardwareInterface with state and command interfaces
- Registered plugin for hardware interface

File: My-ROS2-Humble/Tutorial_ROS2_Control/ROS2Ctrl_ws/install/mobilebot_description/share/mobilebot_description/urdf/arm.xacro (robot description, xacro)
@@ -1 +1,79 @@
-/home/saeedbazargan/Desktop/My-ROS2_Projects/My-ROS2-Humble/Tutorial_ROS2_Control/ROS2Ctrl_ws/src/mobilebot_description/urdf/arm.xacro
+<?xml version="1.0"?>
+<robot xmlns:xacro="http://www.ros.org/wiki/xacro">
+    <!-- #### ##### xacro defines ##### #### -->
+    <xacro:property name="PI"               value="3.14159"/>
+    <xacro:property name="arm_base_length"  value="0.1"/>
+    <xacro:property name="arm_base_width"   value="0.1"/>
+    <xacro:property name="arm_base_height"  value="0.02"/>
+    <xacro:property name="forearm_radius"   value="0.02"/>
+    <xacro:property name="forearm_length"   value="0.3"/>
+    <xacro:property name="hand_radius"      value="0.02"/>
+    <xacro:property name="hand_length"      value="0.3"/>
+    <link name="arm_base_link">
+        <visual>
+            <geometry>
+                <box size="${arm_base_length} ${arm_base_width} ${arm_base_height}"/>
+            </geometry>
+            <origin xyz="0 0 ${arm_base_height/2}" rpy="0 0 0"/>
+            <material name="orange"/>
+        </visual>
+        <collision>
+            <geometry>
+                <box size="${arm_base_length} ${arm_base_width} ${arm_base_height}"/>
+            </geometry>
+            <origin xyz="0 0 ${arm_base_height/2}" rpy="0 0 0"/>
+        </collision>
+        <xacro:box_inertia mass="0.3" length="${arm_base_length}" width="${arm_base_width}" height="${arm_base_height}"
+                           xyz="0 0 ${arm_base_height/2}" rpy="0 0 0"/>
+    </link>
+    <link name="forearm_link">
+        <visual>
+            <geometry>
+                <cylinder radius="${forearm_radius}" length="${forearm_length}"/>
+            </geometry>
+            <origin xyz="0 0 ${forearm_length/2}" rpy="0 0 0"/>
+            <material name="green"/>
+        </visual>
+        <collision>
+            <geometry>
+                <cylinder radius="${forearm_radius}" length="${forearm_length}"/>
+            </geometry>
+            <origin xyz="0 0 ${forearm_length/2}" rpy="0 0 0"/>
+        </collision>
+        <xacro:cylinder_inertia mass="0.2" radius="${forearm_radius}" height="${forearm_length}"
+                           xyz="0 0 ${forearm_length/2}" rpy="0 0 0"/>
+    </link>
+    <joint name="arm_base_forearm_joint" type="revolute">
+        <parent link="arm_base_link"/>
+        <child link="forearm_link"/>
+        <origin xyz="0 0 ${arm_base_height}" rpy="0 0 0"/>
+        <axis xyz="0 1 0"/>
+        <limit lower="0" upper="${PI/2}" effort="100" velocity="100"/>
+        <dynamics friction="0.05" damping="0.1"/>
+    </joint>
+    <link name="hand_link">
+        <visual>
+            <geometry>
+                <cylinder radius="${hand_radius}" length="${hand_length}"/>
+            </geometry>
+            <origin xyz="0 0 ${hand_length/2}" rpy="0 0 0"/>
+            <material name="orange"/>
+        </visual>
+        <collision>
+            <geometry>
+                <cylinder radius="${hand_radius}" length="${hand_length}"/>
+            </geometry>
+            <origin xyz="0 0 ${hand_length/2}" rpy="0 0 0"/>
+        </collision>
+        <xacro:cylinder_inertia mass="0.2" radius="${hand_radius}" height="${hand_length}"
+                           xyz="0 0 ${hand_length/2}" rpy="0 0 0"/>
+    </link>
+    <joint name="forearm_hand_joint" type="revolute">
+        <parent link="forearm_link"/>
+        <child link="hand_link"/>
+        <origin xyz="0 0 ${forearm_length}" rpy="0 0 0"/>
+        <axis xyz="0 1 0"/>
+        <limit lower="0" upper="${PI/2}" effort="100" velocity="100"/>
+        <dynamics friction="0.05" damping="0.1"/>
+    </joint>
+</robot>

File: My-ROS2-Humble/Tutorial_ROS2_Control/ROS2Ctrl_ws/install/mobilebot_description/share/mobilebot_description/urdf/arm_gazebo.xacro (robot description, xacro)
@@ -1 +1,29 @@
-/home/saeedbazargan/Desktop/My-ROS2_Projects/My-ROS2-Humble/Tutorial_ROS2_Control/ROS2Ctrl_ws/src/mobilebot_description/urdf/arm_gazebo.xacro
+<?xml version="1.0"?>
+<robot xmlns:xacro="http://www.ros.org/wiki/xacro">
+    <gazebo reference="arm_base_link">
+        <material>Gazebo/Orange</material>
+    </gazebo>
+    <gazebo reference="forearm_link">
+        <material>Gazebo/Green</material>
+    </gazebo>
+    <gazebo reference="hand_link">
+        <material>Gazebo/Orange</material>
+    </gazebo>
+    <gazebo>
+        <plugin name="joint_state_publisher_controller"
+            filename="libgazebo_ros_joint_state_publisher.so">
+            <!-- Update rate in Hertz -->
+            <update_rate>10</update_rate>
+            <!-- Name of joints in the model whose states will be published. -->
+            <joint_name>arm_base_forearm_joint</joint_name>
+            <joint_name>forearm_hand_joint</joint_name>
+        </plugin>
+    </gazebo>
+    <gazebo>
+        <plugin name="joint_pose_trajectory_controller"
+            filename="libgazebo_ros_joint_pose_trajectory.so">
+            <!-- Update rate in Hz -->
+            <update_rate>2</update_rate>
+        </plugin>
+    </gazebo>
+</robot>

File: My-ROS2-Humble/Tutorial_ROS2_Control/ROS2Ctrl_ws/install/mobilebot_description/share/mobilebot_description/urdf/common_properties.xacro (robot description, xacro)
@@ -1 +1,42 @@
-/home/saeedbazargan/Desktop/My-ROS2_Projects/My-ROS2-Humble/Tutorial_ROS2_Control/ROS2Ctrl_ws/src/mobilebot_description/urdf/common_properties.xacro
+<?xml version="1.0"?>
+<robot xmlns:xacro="http://www.ros.org/wiki/xacro">
+    <material name="green">
+        <color rgba="0 0.5 0 1"/>
+    </material>
+    <material name="blue">
+        <color rgba="0 0 0.5 1"/>
+    </material>
+    <material name="red">
+        <color rgba="0.5 0 0 1"/>
+    </material>
+    <material name="orange">
+        <color rgba="1 0.3 0 1"/>
+    </material>
+    <xacro:macro name="box_inertia" params="mass length width height xyz rpy">
+        <inertial>
+            <origin xyz="${xyz}" rpy="${rpy}"/>
+            <mass value="${mass}"/>
+            <inertia ixx="${(mass/12) * (height*height + length*length)}" ixy="0" ixz="0"
+                     iyy="${(mass/12) * (width*width + length*length)}" iyz="0"
+                     izz="${(mass/12) * (width*width + height*height)}"/>
+        </inertial>
+    </xacro:macro>
+    <xacro:macro name="cylinder_inertia" params="mass radius height xyz rpy">
+        <inertial>
+            <origin xyz="${xyz}" rpy="${rpy}"/>
+            <mass value="${mass}"/>
+            <inertia ixx="${(mass/12) * (3*radius*radius + height*height)}" ixy="0" ixz="0"
+                     iyy="${(mass/12) * (3*radius*radius + height*height)}" iyz="0"
+                     izz="${(mass/2) * (radius*radius)}"/>
+        </inertial>
+    </xacro:macro>
+    <xacro:macro name="sphere_inertia" params="mass radius xyz rpy">
+        <inertial>
+            <origin xyz="${xyz}" rpy="${rpy}"/>
+            <mass value="${mass}"/>
+            <inertia ixx="${(2/5) * mass * radius*radius}" ixy="0" ixz="0"
+                     iyy="${(2/5) * mass * radius*radius}" iyz="0"
+                     izz="${(2/5) * mass * radius*radius}"/>
+        </inertial>
+    </xacro:macro>
+</robot>

File: My-ROS2-Humble/Tutorial_ROS2_Control/ROS2Ctrl_ws/install/mobilebot_description/share/mobilebot_description/urdf/mobilebot.urdf.xacro (robot description, xacro)
@@ -1 +1,16 @@
-/home/saeedbazargan/Desktop/My-ROS2_Projects/My-ROS2-Humble/Tutorial_ROS2_Control/ROS2Ctrl_ws/src/mobilebot_description/urdf/mobilebot.urdf.xacro
+<?xml version="1.0"?>
+<robot name="mobilebot" xmlns:xacro="http://www.ros.org/wiki/xacro">
+    <!-- xacro includes -->
+    <xacro:include filename="common_properties.xacro"/>
+    <xacro:include filename="mobilebot_base.xacro"/>
+    <xacro:include filename="mobilebot_base_gazebo.xacro"/>
+    <xacro:include filename="arm.xacro"/>
+    <xacro:include filename="arm_gazebo.xacro"/>
+    <xacro:include filename="mobilebot_base.ros2_control.xacro"/>
+    <!-- #### Combine the robot(mobilebot) and arm #### -->
+    <joint name="mobilebot_base_arm_joint" type="fixed">
+        <parent link="base_link"/>
+        <child link="arm_base_link"/>
+        <origin xyz="${base_length/4} 0 ${base_height}" rpy="0 0 0"/>
+    </joint>
+</robot>

File: My-ROS2-Humble/Tutorial_ROS2_Control/ROS2Ctrl_ws/install/mobilebot_description/share/mobilebot_description/urdf/mobilebot_base.ros2_control.xacro (robot description, xacro)
@@ -1 +1,31 @@
-/home/saeedbazargan/Desktop/My-ROS2_Projects/My-ROS2-Humble/Tutorial_ROS2_Control/ROS2Ctrl_ws/src/mobilebot_description/urdf/mobilebot_base.ros2_control.xacro
+<?xml version="1.0"?>
+<robot xmlns:xacro="http://www.ros.org/wiki/xacro">
+    <!-- Defines a ROS2 Control hardware interface for the robot.
+        - name: The unique name for this hardware system interface. It can be abc or anything.
+        - type="system": Indicates this is a system-level interface managing multiple joints.
+    -->
+    <ros2_control name="MobileBase" type="system">
+        <hardware>
+            <!-- Here we use a mock plugin for simulation/testing purposes. -->
+            <!-- <plugin>mock_components/GenericSystem</plugin> -->
+            <!-- Enables dynamic calculations for joints (e.g., velocity, position, effort). Useful for more realistic simulations. -->
+            <!-- <param name="calculate_dynamics">true</param> -->
+            <plugin>mobile_base_hardware/MobileBaseHardwareInterface</plugin>
+            <param name="DXL_ID">1</param>
+            <param name="DXL_Port">/dev/ttyUSB0</param>
+        </hardware>
+        <!-- Defines the right wheel joint of the mobile base. -->
+        <joint name="base_RightWheel_joint">
+            <!-- The joint accepts velocity commands (angular velocity for the wheel). -->
+            <command_interface name="velocity" />
+            <!-- he joint reports its position and velocity state -->
+            <state_interface name="position" />
+            <state_interface name="velocity" />
+        </joint>
+        <joint name="base_LeftWheel_joint">
+            <command_interface name="velocity" />
+            <state_interface name="position" />
+            <state_interface name="velocity" />
+        </joint>
+    </ros2_control>
+</robot>

File: My-ROS2-Humble/Tutorial_ROS2_Control/ROS2Ctrl_ws/install/mobilebot_description/share/mobilebot_description/urdf/mobilebot_base.xacro (robot description, xacro)
@@ -1 +1,93 @@
-/home/saeedbazargan/Desktop/My-ROS2_Projects/My-ROS2-Humble/Tutorial_ROS2_Control/ROS2Ctrl_ws/src/mobilebot_description/urdf/mobilebot_base.xacro
+<?xml version="1.0"?>
+<robot xmlns:xacro="http://www.ros.org/wiki/xacro">
+    <!-- #### ##### xacro defines ##### #### -->
+    <xacro:property name="PI"           value="3.14159"/>
+    <xacro:property name="base_length"  value="0.6"/>
+    <xacro:property name="base_width"   value="0.4"/>
+    <xacro:property name="base_height"  value="0.2"/>
+    <xacro:property name="wheel_radius" value="0.1"/>
+    <xacro:property name="wheel_length" value="0.05"/>
+    <!-- #### ##### Base Link and Base footprint ##### #### -->
+    <link name="base_footprint"/>
+    <link name="base_link">
+        <visual>    <!-- give a shape to it -->
+             <geometry>
+                <box size="${base_length} ${base_width} ${base_height}"/>   <!-- 60cm length, 40cm width, 20cm height-->
+             </geometry>
+             <origin xyz="0 0 ${base_height/2}" rpy="0 0 0"/>
+             <material name="blue"/>
+        </visual>
+        <collision>
+            <geometry>
+                <box size="${base_length} ${base_width} ${base_height}"/>   <!-- 60cm length, 40cm width, 20cm height-->
+             </geometry>
+             <origin xyz="0 0 ${base_height/2}" rpy="0 0 0"/>
+        </collision>
+        <xacro:box_inertia mass="1.0" length="${base_length}" width="${base_width}" height="${base_height}"
+                            xyz="0 0 ${base_height/2}" rpy="0 0 0"/>
+    </link>
+    <joint name="footprint_BaseLink_joint" type="fixed">
+        <parent link="base_footprint"/>
+        <child link="base_link"/>
+        <origin xyz="0 0 ${wheel_radius}" rpy="0 0 0"/>
+    </joint>
+    <!-- #### ##### xacro functions ##### #### -->
+    <xacro:macro name="wheel_link" params="prefix">
+        <link name="${prefix}_wheel_link">
+            <visual>
+                <geometry>
+                    <cylinder radius="${wheel_radius}" length="${wheel_length}"/>
+                </geometry>
+                <origin xyz="0 0 0" rpy="${PI/2} 0 0"/>     <!-- 90degree in X-Axis-->
+                <material name="red"/>
+            </visual>
+            <collision>
+                <geometry>
+                    <cylinder radius="${wheel_radius}" length="${wheel_length}"/>
+                </geometry>
+                <origin xyz="0 0 0" rpy="${PI/2} 0 0"/>     <!-- 90degree in X-Axis-->
+            </collision>
+            <xacro:cylinder_inertia mass="0.4" radius="${wheel_radius}" height="${wheel_length}"
+                                     xyz="0 0 0" rpy="${PI/2} 0 0"/>
+        </link>
+    </xacro:macro>
+    <!-- #### ##### Right Wheel Link ##### #### -->
+    <xacro:wheel_link prefix="right"/>
+    <joint name="base_RightWheel_joint" type="continuous">  <!-- continuous is a revolution with no limit-->
+        <parent link="base_link"/>
+        <child link="right_wheel_link"/>
+        <origin xyz="-${base_length/4} -${(base_width + wheel_length) / 2} 0" rpy="0 0 0"/>     <!-- 15cm: pulled back, 22.5cm: pulled right-->
+        <axis xyz="0 1 0"/> <!-- rotate on Y-Axis -->
+    </joint>
+    <!-- #### ##### Left Wheel Link ##### #### -->
+    <xacro:wheel_link prefix="left"/>
+    <joint name="base_LeftWheel_joint" type="continuous">  <!-- continuous is a revolution with no limit-->
+        <parent link="base_link"/>
+        <child link="left_wheel_link"/>
+        <origin xyz="-${base_length/4} ${(base_width + wheel_length) / 2} 0" rpy="0 0 0"/>     <!-- 15cm: pulled back, 22.5cm: pulled left-->
+        <axis xyz="0 1 0"/> <!-- rotate on Y-Axis -->
+    </joint>
+    <!-- #### ##### Caster Wheel Link ##### #### -->
+    <link name="caster_wheel_link">
+        <visual>
+            <geometry>
+                <sphere radius="${wheel_radius/2}"/>
+            </geometry>
+            <origin xyz="0 0 0" rpy="0 0 0"/>
+            <material name="red"/>
+        </visual>
+        <collision>
+            <geometry>
+                <sphere radius="${wheel_radius/2}"/>
+            </geometry>
+            <origin xyz="0 0 0" rpy="0 0 0"/>
+        </collision>
+        <xacro:sphere_inertia mass="0.2" radius="${wheel_radius/2}"
+                              xyz="0 0 0" rpy="0 0 0"/>
+    </link>
+    <joint name="base_CasterWheel_joint" type="fixed">
+        <parent link="base_link"/>
+        <child link="caster_wheel_link"/>
+        <origin xyz="${base_length/3} 0 -${wheel_radius/2}" rpy="0 0 0"/>
+    </joint>
+</robot>

File: My-ROS2-Humble/Tutorial_ROS2_Control/ROS2Ctrl_ws/install/mobilebot_description/share/mobilebot_description/urdf/mobilebot_base_gazebo.xacro (robot description, xacro)
@@ -1 +1,38 @@
-/home/saeedbazargan/Desktop/My-ROS2_Projects/My-ROS2-Humble/Tutorial_ROS2_Control/ROS2Ctrl_ws/src/mobilebot_description/urdf/mobilebot_base_gazebo.xacro
+<?xml version="1.0"?>
+<robot xmlns:xacro="http://www.ros.org/wiki/xacro">
+    <!-- #### ##### everything I write in this gazebo tag will apply to the base_link -->
+    <gazebo reference="base_link">
+        <material>Gazebo/Blue</material>
+    </gazebo>
+    <gazebo reference="right_wheel_link">
+        <material>Gazebo/Red</material>
+    </gazebo>
+    <gazebo reference="left_wheel_link">
+        <material>Gazebo/Red</material>
+    </gazebo>
+    <gazebo reference="caster_wheel_link">
+        <material>Gazebo/Red</material>
+        <mu1 value="0.1"/>
+        <mu2 value="0.1"/>
+    </gazebo>
+    <!-- #### Gazebo Plugins ##### -->
+    <gazebo>
+        <plugin name="diff_drive_controller" filename="libgazebo_ros_diff_drive.so">
+            <!-- Update rate in Hz -->
+            <update_rate>50</update_rate>
+            <!-- wheels -->
+            <left_joint>base_LeftWheel_joint</left_joint>
+            <right_joint>base_RightWheel_joint</right_joint>
+            <!-- kinematics -->
+            <wheel_separation>0.45</wheel_separation>
+            <wheel_diameter>0.2</wheel_diameter>
+            <!-- output -->
+            <publish_odom>true</publish_odom>
+            <publish_odom_tf>true</publish_odom_tf>
+            <publish_wheel_tf>true</publish_wheel_tf>
+            <odometry_topic>odom</odometry_topic>
+            <odometry_frame>odom</odometry_frame>
+            <robot_base_frame>base_footprint</robot_base_frame>
+        </plugin>
+    </gazebo>
+</robot>

File: My-ROS2-Humble/Tutorial_ROS2_Control/ROS2Ctrl_ws/install/mobilebot_description/share/mobilebot_description/urdf/standalone_arm.urdf.xacro (robot description, xacro)
@@ -1 +1,6 @@
-/home/saeedbazargan/Desktop/My-ROS2_Projects/My-ROS2-Humble/Tutorial_ROS2_Control/ROS2Ctrl_ws/src/mobilebot_description/urdf/standalone_arm.urdf.xacro
+<?xml version="1.0"?>
+<robot name="mobilebot" xmlns:xacro="http://www.ros.org/wiki/xacro">
+    <xacro:include filename="common_properties.xacro"/>
+    <xacro:include filename="arm.xacro"/>
+    <xacro:include filename="arm_gazebo.xacro"/>
+</robot>

File: My-ROS2-Humble/Tutorial_ROS2_Control/ROS2Ctrl_ws/src/mobilebot_description/urdf/mobilebot.urdf.xacro (robot description, xacro)
@@ -4,13 +4,14 @@
     <xacro:include filename="common_properties.xacro"/>
     <xacro:include filename="mobilebot_base.xacro"/>
-    <!-- <xacro:include filename="mobilebot_base_gazebo.xacro"/>
+    <xacro:include filename="mobilebot_base_gazebo.xacro"/>
     <xacro:include filename="arm.xacro"/>
-    <xacro:include filename="arm_gazebo.xacro"/> -->
+    <xacro:include filename="arm_gazebo.xacro"/>
     <xacro:include filename="mobilebot_base.ros2_control.xacro"/>
+    <xacro:include filename="arm.ros2_control.xacro"/>
     <!-- #### Combine the robot(mobilebot) and arm #### -->
-    <!-- <joint name="mobilebot_base_arm_joint" type="fixed">
+    <joint name="mobilebot_base_arm_joint" type="fixed">
         <parent link="base_link"/>
         <child link="arm_base_link"/>
         <origin xyz="${base_length/4} 0 ${base_height}" rpy="0 0 0"/>
-    </joint> -->
+    </joint>
 </robot>

File: My-ROS2-Humble/Tutorial_ROS2_Control/ROS2Ctrl_ws/src/mobilebot_description/urdf/mobilebot_base.ros2_control.xacro (robot description, xacro)
@@ -2,8 +2,8 @@
 <robot xmlns:xacro="http://www.ros.org/wiki/xacro">
     <!-- Defines a ROS2 Control hardware interface for the robot.
-        - name: The unique name for this hardware system interface.
+        - name: The unique name for this hardware system interface. It can be abc or anything.
         - type="system": Indicates this is a system-level interface managing multiple joints.
     -->
-    <ros2_control name="MobileBaseHardwareInterface" type="system">
+    <ros2_control name="MobileBase" type="system">
         <hardware>
             <!-- Here we use a mock plugin for simulation/testing purposes. -->
@@ -11,4 +11,5 @@
             <!-- Enables dynamic calculations for joints (e.g., velocity, position, effort). Useful for more realistic simulations. -->
             <param name="calculate_dynamics">true</param>
+            <!-- <plugin>mobile_base_hardware/MobileBaseHardwareInterface</plugin> -->
         </hardware>
         <!-- Defines the right wheel joint of the mobile base. -->
@@ -16,5 +17,5 @@
             <!-- The joint accepts velocity commands (angular velocity for the wheel). -->
             <command_interface name="velocity" />
-            <!-- he joint reports its position and velocity state -->
+            <!-- The joint reports its position and velocity state -->
             <state_interface name="position" />
             <state_interface name="velocity" />
