Commit message: Launch file modified.

File: My-ROS2-Humble/Kukabot_MobileRobot/kukabot_ws/src/kukabot_description/urdf/kukabot_wheel.xacro (robot description, xacro)
@@ -2,6 +2,6 @@
 <robot xmlns:xacro="http://www.ros.org/wiki/xacro">
 <!-- ##################################################################################################### -->
-    <xacro:macro name="kukawheel" params="prefix">
-        <link name="wheel_link_${prefix}">
+    <xacro:macro name="kukawheel">
+        <link name="wheel_link_frontLeft">
             <visual>
                 <geometry>
@@ -26,7 +26,106 @@
             </inertial>
         </link>
-        <joint name="wheel_joint_${prefix}" type="continuous">
-            <parent link="caster_link_${prefix}"/>
-            <child link="wheel_link_${prefix}"/>
+        <joint name="wheel_joint_frontLeft" type="continuous">
+            <parent link="caster_link_frontLeft"/>
+            <child link="wheel_link_frontLeft"/>
+            <origin xyz="${wheel_offset_x} ${wheel_offset_y} ${wheel_offset_z}" rpy="0 0 0"/>
+            <axis xyz="0 1 0"/>
+            <limit effort="${wheel_joint_effort}" velocity="${wheel_joint_velocity}"/>
+            <dynamics damping="${wheel_joint_damping}" friction="${wheel_joint_friction}"/>
+            <safety_controller k_velocity="${wheel_joint_safety_k_velocity}"/>
+        </joint>
+<!-- ##################################################################################################### -->
+        <link name="wheel_link_frontRight">
+            <visual>
+                <geometry>
+                    <mesh filename="package://kukabot_description/meshes/base/front-right_wheel.dae" />
+                    <!-- <sphere radius="${wheel_radius}"/> -->
+                </geometry>
+                <origin xyz="0 0 0" rpy="0 0 0"/>
+                <material name="Orange"/>
+            </visual>
+            <collision>
+                <geometry>
+                    <cylinder radius="${wheel_radius}" length="${wheel_radius}"/>
+                </geometry>
+                <origin xyz="0 0 0" rpy="${M_PI/2} 0 0"/>
+            </collision>
+            <inertial>
+                <mass value="${wheel_mass}"/>
+                <origin xyz="0 0 0"/>
+                <inertia ixx="0.012411765597" ixy="-0.000711733678" ixz="0.00050272983"
+                         iyy="0.015218160428" iyz="-0.000004273467"
+                         izz="0.011763977943"/>
+            </inertial>
+        </link>
+        <joint name="wheel_joint_frontRight" type="continuous">
+            <parent link="caster_link_frontRight"/>
+            <child link="wheel_link_frontRight"/>
+            <origin xyz="${wheel_offset_x} ${wheel_offset_y} ${wheel_offset_z}" rpy="0 0 0"/>
+            <axis xyz="0 1 0"/>
+            <limit effort="${wheel_joint_effort}" velocity="${wheel_joint_velocity}"/>
+            <dynamics damping="${wheel_joint_damping}" friction="${wheel_joint_friction}"/>
+            <safety_controller k_velocity="${wheel_joint_safety_k_velocity}"/>
+        </joint>
+<!-- ##################################################################################################### -->
+        <link name="wheel_link_backLeft">
+            <visual>
+                <geometry>
+                    <mesh filename="package://kukabot_description/meshes/base/back-left_wheel.dae" />
+                    <!-- <sphere radius="${wheel_radius}"/> -->
+                </geometry>
+                <origin xyz="0 0 0" rpy="0 0 0"/>
+                <material name="Orange"/>
+            </visual>
+            <collision>
+                <geometry>
+                    <cylinder radius="${wheel_radius}" length="${wheel_radius}"/>
+                </geometry>
+                <origin xyz="0 0 0" rpy="${M_PI/2} 0 0"/>
+            </collision>
+            <inertial>
+                <mass value="${wheel_mass}"/>
+                <origin xyz="0 0 0"/>
+                <inertia ixx="0.012411765597" ixy="-0.000711733678" ixz="0.00050272983"
+                         iyy="0.015218160428" iyz="-0.000004273467"
+                         izz="0.011763977943"/>
+            </inertial>
+        </link>
+        <joint name="wheel_joint_backLeft" type="continuous">
+            <parent link="caster_link_backLeft"/>
+            <child link="wheel_link_backLeft"/>
+            <origin xyz="${wheel_offset_x} ${wheel_offset_y} ${wheel_offset_z}" rpy="0 0 0"/>
+            <axis xyz="0 1 0"/>
+            <limit effort="${wheel_joint_effort}" velocity="${wheel_joint_velocity}"/>
+            <dynamics damping="${wheel_joint_damping}" friction="${wheel_joint_friction}"/>
+            <safety_controller k_velocity="${wheel_joint_safety_k_velocity}"/>
+        </joint>
+<!-- ##################################################################################################### -->
+        <link name="wheel_link_backRight">
+            <visual>
+                <geometry>
+                    <mesh filename="package://kukabot_description/meshes/base/back-right_wheel.dae" />
+                    <!-- <sphere radius="${wheel_radius}"/> -->
+                </geometry>
+                <origin xyz="0 0 0" rpy="0 0 0"/>
+                <material name="Orange"/>
+            </visual>
+            <collision>
+                <geometry>
+                    <cylinder radius="${wheel_radius}" length="${wheel_radius}"/>
+                </geometry>
+                <origin xyz="0 0 0" rpy="${M_PI/2} 0 0"/>
+            </collision>
+            <inertial>
+                <mass value="${wheel_mass}"/>
+                <origin xyz="0 0 0"/>
+                <inertia ixx="0.012411765597" ixy="-0.000711733678" ixz="0.00050272983"
+                         iyy="0.015218160428" iyz="-0.000004273467"
+                         izz="0.011763977943"/>
+            </inertial>
+        </link>
+        <joint name="wheel_joint_backRight" type="continuous">
+            <parent link="caster_link_backRight"/>
+            <child link="wheel_link_backRight"/>
             <origin xyz="${wheel_offset_x} ${wheel_offset_y} ${wheel_offset_z}" rpy="0 0 0"/>
             <axis xyz="0 1 0"/>

File: My-ROS2-Humble/Kukabot_MobileRobot/kukabot_ws/src/kukabot_description/urdf/main.gazebo.xacro (robot description, xacro)
@@ -5,5 +5,5 @@
         <gazebo>
             <plugin filename="gz_ros2_control-system" name="gz_ros2_control::GazeboSimROS2ControlPlugin">
-                <parameters>$(find kukabot_bringup)/config/kukabot_sim.yaml</parameters>
+                <parameters>$(find kukabot_bringup)/config/kukabot_sim_controller.yaml</parameters>
             </plugin>
         </gazebo>

File: My-ROS2-Humble/Kukabot_MobileRobot/kukabot_ws/src/kukabot_description/urdf/main.ros2_control.xacro (robot description, xacro)
@@ -15,4 +15,28 @@
                 <state_interface name="velocity"/>
             </joint>
+            <joint name="wheel_joint_frontRight">
+                <command_interface name="velocity">
+                    <param name="min">-1</param>
+                    <param name="max">1</param>
+                </command_interface>
+                <state_interface name="position"/>
+                <state_interface name="velocity"/>
+            </joint>
+            <joint name="wheel_joint_backLeft">
+                <command_interface name="velocity">
+                    <param name="min">-1</param>
+                    <param name="max">1</param>
+                </command_interface>
+                <state_interface name="position"/>
+                <state_interface name="velocity"/>
+            </joint>
+            <joint name="wheel_joint_backRight">
+                <command_interface name="velocity">
+                    <param name="min">-1</param>
+                    <param name="max">1</param>
+                </command_interface>
+                <state_interface name="position"/>
+                <state_interface name="velocity"/>
+            </joint>
         </ros2_control>
     </xacro:macro>

File: My-ROS2-Humble/Kukabot_MobileRobot/kukabot_ws/src/kukabot_description/urdf/main.urdf.xacro (robot description, xacro)
@@ -15,5 +15,5 @@
     <xacro:kukabase                 name="base"/>
     <xacro:kukacaster               name="base"/>
-    <xacro:kukawheel                prefix="frontLeft"/>
+    <xacro:kukawheel/>
     <!-- Base -->
     <xacro:kukabase_gazebo/>
@@ -25,4 +25,7 @@
     <!-- Wheel -->
     <xacro:kukawheel_gazebo         prefix="frontLeft"/>
+    <xacro:kukawheel_gazebo         prefix="frontRight"/>
+    <xacro:kukawheel_gazebo         prefix="backLeft"/>
+    <xacro:kukawheel_gazebo         prefix="backRight"/>
     <xacro:main_gazebo/>
     <xacro:main_ros2_control/>
