Commit message: feat(camera): add Gazebo camera sensor to robot
- Add camera link and fixed joint to the robot
- Add simplified camera sensor for gz-sim
- Configure image topic, resolution, FOV, and update rate
- Use OGRE2 as the Gazebo rendering engine

File: My-ROS2/Omni4Wheel_MobileRobot/omni_ws/src/omnirobot_description/urdf/gazebo.xacro (robot description, xacro)
@@ -2,4 +2,7 @@
 <robot xmlns:xacro="http://www.ros.org/wiki/xacro">
     <gazebo reference="base_link">
+        <material>Gazebo/Blue</material>
+    </gazebo>
+    <gazebo reference="l_Body001">
         <material>Gazebo/Blue</material>
     </gazebo>

File: My-ROS2/Omni4Wheel_MobileRobot/omni_ws/src/omnirobot_description/urdf/gazebo_ros2_control.xacro (robot description, xacro)
@@ -4,4 +4,5 @@
     <xacro:include filename="$(find omnirobot_description)/urdf/common_properties.xacro"/>
     <xacro:include filename="$(find omnirobot_description)/urdf/base.xacro"/>
+    <xacro:include filename="$(find omnirobot_description)/urdf/camera.xacro"/>
     <xacro:include filename="$(find omnirobot_description)/urdf/gazebo.xacro"/>
     <ros2_control name="omnirobot_gazebo" type="system">

File: My-ROS2/Omni4Wheel_MobileRobot/omni_ws/src/omnirobot_description/urdf/main.xacro (robot description, xacro)
@@ -4,4 +4,5 @@
     <xacro:include filename="$(find omnirobot_description)/urdf/common_properties.xacro"/>
     <xacro:include filename="$(find omnirobot_description)/urdf/base.xacro"/>
+    <xacro:include filename="$(find omnirobot_description)/urdf/camera.xacro"/>
     <xacro:include filename="$(find omnirobot_description)/urdf/gazebo.xacro"/>
     <xacro:include filename="$(find omnirobot_description)/urdf/ros2_control.xacro"/>
